Commit message: model urdf shown in rviz and gazebo

File: robot_v3/urdf/model.urdf (robot description, URDF)
Before this commit: robot robot_v2, 16 links, 15 joints
Links:
- link base_link: geometry collision mesh filename=package://robot_v3/meshes/base_link.STL; visual mesh filename=package://robot_v3/meshes/base_link.STL
- link link_1: geometry collision mesh filename=package://robot_v3/meshes/link_1.STL; visual mesh filename=package://robot_v3/meshes/link_1.STL
- link link_2: geometry collision mesh filename=package://robot_v3/meshes/link_2.STL; visual mesh filename=package://robot_v3/meshes/link_2.STL
- link link_3: geometry collision mesh filename=package://robot_v3/meshes/link_3.STL; visual mesh filename=package://robot_v3/meshes/link_3.STL
- link link_4: geometry collision mesh filename=package://robot_v3/meshes/link_4.STL; visual mesh filename=package://robot_v3/meshes/link_4.STL
- link pre_link_5: geometry collision mesh filename=package://robot_v3/meshes/pre_link_5.STL; visual mesh filename=package://robot_v3/meshes/pre_link_5.STL
- link wheel_link_1: geometry collision mesh filename=package://robot_v3/meshes/wheel_link_1.STL; visual mesh filename=package://robot_v3/meshes/wheel_link_1.STL
- link wheel_link_2: geometry collision mesh filename=package://robot_v3/meshes/wheel_link_2.STL; visual mesh filename=package://robot_v3/meshes/wheel_link_2.STL
- link wheel_link_3: geometry collision mesh filename=package://robot_v3/meshes/wheel_link_3.STL; visual mesh filename=package://robot_v3/meshes/wheel_link_3.STL
- link wheel_link_4: geometry collision mesh filename=package://robot_v3/meshes/wheel_link_4.STL; visual mesh filename=package://robot_v3/meshes/wheel_link_4.STL

Commit message: adjusted gripper position

File: robot_v3/urdf/model.urdf (robot description, URDF)
Before this commit: robot robot_v3, 16 links, 15 joints
Joints:
- joint joint_gripper: origin xyz=0 0 0.07 rpy=0 0 0 -> xyz=0.015 -0.015 0.015 rpy=-1.571 -2.071 -3.141

Commit message: aruco tag visible

File: robot_v3/urdf/model.urdf (robot description, URDF)
Before this commit: robot robot_v3, 16 links, 15 joints
Links:
- added link aruco_link, mass 8.1643; collision box size=0.1 0.1 0.001; visual box size=0.1 0.1 0.001
- link base_link: geometry collision mesh filename=package://robot_v3/meshes/base_link.STL; visual box size=0.12 0.12 0.0004
Joints:
- added joint joint_aruco_tag: type fixed, parent base_link, child aruco_link, origin xyz=0.0 -0.22 0.051 rpy=0 0 0

Commit message: new robot seeing in gazebo but not rviz2

File: robot_v3/urdf/model.urdf (robot description, URDF)
Before this commit: robot robot_v3, 17 links, 16 joints
Links:
- link base_link: geometry collision mesh filename=file://meshes/base_link.STL; visual box size=0.12 0.12 0.0004
- link gripper_actuactor_link: geometry collision mesh filename=file://meshes/actuactor_link.STL; visual mesh filename=file://meshes/actuactor_link.STL
- link gripper_arm_1_link: geometry collision mesh filename=file://meshes/arm_1_link.STL; visual mesh filename=file://meshes/arm_1_link.STL
- link gripper_arm_2_link: geometry collision mesh filename=file://meshes/arm_2_link.STL; visual mesh filename=file://meshes/arm_2_link.STL
- link gripper_base_link: geometry collision mesh filename=file://meshes/gripper_base_link.STL; visual mesh filename=file://meshes/gripper_base_link.STL
- link gripper_shaft_1_link: geometry collision mesh filename=file://meshes/shaft_1_link.STL; visual mesh filename=file://meshes/shaft_1_link.STL
- link gripper_shaft_2_link: geometry collision mesh filename=file://meshes/shaft_2_link.STL; visual mesh filename=file://meshes/shaft_2_link.STL
- link link_1: geometry collision mesh filename=file://meshes/link_1.STL; visual mesh filename=file://meshes/link_1.STL
- link link_2: geometry collision mesh filename=file://meshes/link_2.STL; visual mesh filename=file://meshes/link_2.STL
- link link_3: geometry collision mesh filename=file://meshes/link_3.STL; visual mesh filename=file://meshes/link_3.STL
- link link_4: geometry collision mesh filename=file://meshes/link_4.STL; visual mesh filename=file://meshes/link_4.STL
- link pre_link_5: geometry collision mesh filename=file://meshes/pre_link_5.STL; visual mesh filename=file://meshes/pre_link_5.STL
- link wheel_link_1: geometry collision mesh filename=file://meshes/wheel_link_1.STL; visual mesh filename=file://meshes/wheel_link_1.STL
- link wheel_link_2: geometry collision mesh filename=file://meshes/wheel_link_2.STL; visual mesh filename=file://meshes/wheel_link_2.STL
- link wheel_link_3: geometry collision mesh filename=file://meshes/wheel_link_3.STL; visual mesh filename=file://meshes/wheel_link_3.STL
- link wheel_link_4: geometry collision mesh filename=file://meshes/wheel_link_4.STL; visual mesh filename=file://meshes/wheel_link_4.STL
Joints:
- joint joint_2: origin xyz=0 -0.024358 0.0098714 rpy=-3.1416 0 3.1416 -> xyz=0 -0.024358 0.0098714 rpy=-1.5708 0 3.1416
- joint joint_3: origin xyz=0 -0.13432 0 rpy=-1.5708 0 0 -> xyz=0 -0.13432 0 rpy=3.1416 0 0
- joint wheel_joint_4: origin xyz=0.0765 -0.054318 0.0060186 rpy=1.5708 1.179 1.5708 -> xyz=0.0765 -0.25731 -0.0032237 rpy=1.5708 1.179 1.5708

File: robot_v3/urdf/ros_robot_v3.urdf (robot description, URDF)
Before this commit: robot ros_robot_v3, 10 links, 9 joints
Links:
- link base_link: mass 8.1643 -> 3.1643
- link link_1: mass 0 -> 0.064021
Joints:
- joint joint_1: limit lower=-3.1415 upper=3.1415 effort=100 velocity=5 -> (none)
- joint joint_2: limit lower=-3.1415 upper=3.1415 effort=100 velocity=5 -> (none); origin xyz=0 -0.024358 0.0098714 rpy=-3.1416 0 3.1416 -> xyz=0 -0.024358 0.0098714 rpy=-1.5708 0 3.1416
- joint joint_3: limit lower=-3.1415 upper=3.1415 effort=100 velocity=5 -> (none); origin xyz=0 -0.13432 0 rpy=-1.5708 0 0 -> xyz=0 -0.13432 0 rpy=3.1416 0 0
- joint joint_4: limit lower=-3.1415 upper=3.1415 effort=100 velocity=5 -> (none)
- joint joint_5: limit lower=-3.1415 upper=3.1415 effort=100 velocity=5 -> (none); origin xyz=-0.0059717 -0.027674 0.056246 rpy=-1.5708 0 0.59278 -> xyz=-0.00060377 0.00065019 0.063746 rpy=-1.5708 0 0.59278
- joint wheel_joint_1: limit lower=-1.79769E+308 upper=-1.79769E+308 effort=100 velocity=10 -> (none)
- joint wheel_joint_2: limit lower=-1.79769E+308 upper=-1.79769E+308 effort=100 velocity=10 -> (none)
- joint wheel_joint_3: limit lower=-1.79769E+308 upper=1.79769E+308 effort=100 velocity=10 -> (none)
- joint wheel_joint_4: limit lower=-1.79769E+308 upper=1.79769E+308 effort=100 velocity=10 -> (none); origin xyz=0.0765 -0.054318 0.0060186 rpy=1.5708 1.179 1.5708 -> xyz=0.0765 -0.25731 -0.0032237 rpy=1.5708 1.179 1.5708

Commit message: arm_commander working fine
no trajectory planner

File: robot_v3/urdf/model.urdf (robot description, URDF)
Before this commit: robot robot_v3, 17 links, 16 joints
Links:
- removed link gripper_actuactor_link
- removed link gripper_arm_1_link
- removed link gripper_arm_2_link
- removed link gripper_base_link
- removed link gripper_shaft_1_link
- removed link gripper_shaft_2_link
Joints:
- removed joint gripper_actuactor_joint
- removed joint gripper_arm_1_joint
- removed joint gripper_arm_2_joint
- removed joint gripper_shaft_1_joint
- removed joint gripper_shaft_2_joint
- removed joint joint_gripper
- joint joint_5: origin xyz=-0.0059717 -0.027674 0.056246 rpy=-1.5708 0 0.59278 -> xyz=-0.00060377 0.00065019 0.063746 rpy=-1.5708 0 0.59278
- joint wheel_joint_1: limit lower=-1.79769E+308 upper=-1.79769E+308 effort=100 velocity=10 -> lower=-1.79769E+308 upper=1.79769E+308 effort=100 velocity=10
- joint wheel_joint_2: limit lower=-1.79769E+308 upper=-1.79769E+308 effort=100 velocity=10 -> lower=-1.79769E+308 upper=1.79769E+308 effort=100 velocity=10

Commit message: add mecanum wheels. Good looking wheel positioning

File: robot_v3/urdf/model.urdf (robot description, URDF)
Before this commit: robot robot_v3, 11 links, 10 joints
Links:
- added link mecanum_link_1_1, mass 0.00323221921166528; collision mesh filename=file://meshes/mecanum_link_1_1.STL; visual mesh filename=file://meshes/mecanum_link_1_1.STL
- added link mecanum_link_1_2, mass 0.00323221921166528; collision mesh filename=file://meshes/mecanum_link_1_2.STL; visual mesh filename=file://meshes/mecanum_link_1_2.STL
- added link mecanum_link_1_3, mass 0.00323221921166513; collision mesh filename=file://meshes/mecanum_link_1_3.STL; visual mesh filename=file://meshes/mecanum_link_1_3.STL
- added link mecanum_link_1_4, mass 0.00323221921166558; collision mesh filename=file://meshes/mecanum_link_1_4.STL; visual mesh filename=file://meshes/mecanum_link_1_4.STL
- added link mecanum_link_1_5, mass 0.00323221921166528; collision mesh filename=file://meshes/mecanum_link_1_5.STL; visual mesh filename=file://meshes/mecanum_link_1_5.STL
- added link mecanum_link_1_6, mass 0.00323221921166558; collision mesh filename=file://meshes/mecanum_link_1_6.STL; visual mesh filename=file://meshes/mecanum_link_1_6.STL
- added link mecanum_link_1_7, mass 0.00323221921166528; collision mesh filename=file://meshes/mecanum_link_1_7.STL; visual mesh filename=file://meshes/mecanum_link_1_7.STL
- added link mecanum_link_1_8, mass 0.00323221921166559; collision mesh filename=file://meshes/mecanum_link_1_8.STL; visual mesh filename=file://meshes/mecanum_link_1_8.STL
- added link mecanum_link_2_1, mass 0.00323221921166513; collision mesh filename=file://meshes/mecanum_link_2_1.STL; visual mesh filename=file://meshes/mecanum_link_2_1.STL
- added link mecanum_link_2_2, mass 0.00323221921166528; collision mesh filename=file://meshes/mecanum_link_2_2.STL; visual mesh filename=file://meshes/mecanum_link_2_2.STL
- added link mecanum_link_2_3, mass 0.00323221921166573; collision mesh filename=file://meshes/mecanum_link_2_3.STL; visual mesh filename=file://meshes/mecanum_link_2_3.STL
- added link mecanum_link_2_4, mass 0.00323221921166512; collision mesh filename=file://meshes/mecanum_link_2_4.STL; visual mesh filename=file://meshes/mecanum_link_2_4.STL
- added link mecanum_link_2_5, mass 0.00323221921166528; collision mesh filename=file://meshes/mecanum_link_2_5.STL; visual mesh filename=file://meshes/mecanum_link_2_5.STL
- added link mecanum_link_2_6, mass 0.00323221921166527; collision mesh filename=file://meshes/mecanum_link_2_6.STL; visual mesh filename=file://meshes/mecanum_link_2_6.STL
- added link mecanum_link_2_7, mass 0.00323221921166513; collision mesh filename=file://meshes/mecanum_link_2_7.STL; visual mesh filename=file://meshes/mecanum_link_2_7.STL
- added link mecanum_link_2_8, mass 0.00323221921166528; collision mesh filename=file://meshes/mecanum_link_2_8.STL; visual mesh filename=file://meshes/mecanum_link_2_8.STL
- added link mecanum_link_3_1, mass 0.00323221921166527; collision mesh filename=file://meshes/mecanum_link_3_1.STL; visual mesh filename=file://meshes/mecanum_link_3_1.STL
- added link mecanum_link_3_2, mass 0.00323221921166513; collision mesh filename=file://meshes/mecanum_link_3_2.STL; visual mesh filename=file://meshes/mecanum_link_3_2.STL
- added link mecanum_link_3_3, mass 0.00323221921166528; collision mesh filename=file://meshes/mecanum_link_3_3.STL; visual mesh filename=file://meshes/mecanum_link_3_3.STL
- added link mecanum_link_3_4, mass 0.00323221921166543; collision mesh filename=file://meshes/mecanum_link_3_4.STL; visual mesh filename=file://meshes/mecanum_link_3_4.STL
- added link mecanum_link_3_5, mass 0.00323221921166543; collision mesh filename=file://meshes/mecanum_link_3_5.STL; visual mesh filename=file://meshes/mecanum_link_3_5.STL
- added link mecanum_link_3_6, mass 0.00323221921166513; collision mesh filename=file://meshes/mecanum_link_3_6.STL; visual mesh filename=file://meshes/mecanum_link_3_6.STL
- added link mecanum_link_3_7, mass 0.00323221921166543; collision mesh filename=file://meshes/mecanum_link_3_7.STL; visual mesh filename=file://meshes/mecanum_link_3_7.STL
- added link mecanum_link_3_8, mass 0.00323221921166528; collision mesh filename=file://meshes/mecanum_link_3_8.STL; visual mesh filename=file://meshes/mecanum_link_3_8.STL
- added link mecanum_link_4_1, mass 0.00323221921166573; collision mesh filename=file://meshes/mecanum_link_4_1.STL; visual mesh filename=file://meshes/mecanum_link_4_1.STL
- added link mecanum_link_4_2, mass 0.00323221921166528; collision mesh filename=file://meshes/mecanum_link_4_2.STL; visual mesh filename=file://meshes/mecanum_link_4_2.STL
- added link mecanum_link_4_3, mass 0.00323221921166528; collision mesh filename=file://meshes/mecanum_link_4_3.STL; visual mesh filename=file://meshes/mecanum_link_4_3.STL
- added link mecanum_link_4_4, mass 0.00323221921166543; collision mesh filename=file://meshes/mecanum_link_4_4.STL; visual mesh filename=file://meshes/mecanum_link_4_4.STL
- added link mecanum_link_4_5, mass 0.00323221921166512; collision mesh filename=file://meshes/mecanum_link_4_5.STL; visual mesh filename=file://meshes/mecanum_link_4_5.STL
- added link mecanum_link_4_6, mass 0.00323221921166513; collision mesh filename=file://meshes/mecanum_link_4_6.STL; visual mesh filename=file://meshes/mecanum_link_4_6.STL
- added link mecanum_link_4_7, mass 0.00323221921166528; collision mesh filename=file://meshes/mecanum_link_4_7.STL; visual mesh filename=file://meshes/mecanum_link_4_7.STL
- added link mecanum_link_4_8, mass 0.00323221921166528; collision mesh filename=file://meshes/mecanum_link_4_8.STL; visual mesh filename=file://meshes/mecanum_link_4_8.STL
- link wheel_link_1: mass 0.13047 -> 0.0979999262042874
- link wheel_link_2: mass 0.13047 -> 0.0959057923631772
- link wheel_link_3: mass 0.13047 -> 0.0959057923631772
- link wheel_link_4: mass 0.13047 -> 0.0979999262042875
Joints:
- added joint mecanum_joint_1_1: type continuous, parent wheel_link_1, child mecanum_link_1_1, origin xyz=-0.02392 -0.010659 -0.0088452 rpy=3.0576 0.5236 -0.95532, axis 1 0 0
- added joint mecanum_joint_1_2: type continuous, parent wheel_link_1, child mecanum_link_1_2, origin xyz=-0.010659 -0.010659 -0.023168 rpy=-1.6479 0 -0.7854, axis 1 0 0
- added joint mecanum_joint_1_3: type continuous, parent wheel_link_1, child mecanum_link_1_3, origin xyz=0.0088452 -0.010659 -0.02392 rpy=1.9316 -0.5236 -0.95532, axis 1 0 0
- added joint mecanum_joint_1_4: type continuous, parent wheel_link_1, child mecanum_link_1_4, origin xyz=0.023168 -0.010659 -0.010659 rpy=0.19357 -0.7854 -1.5708, axis 1 0 0
- added joint mecanum_joint_1_5: type continuous, parent wheel_link_1, child mecanum_link_1_5, origin xyz=0.02392 -0.010659 0.0088452 rpy=-2.5986 -0.5236 -2.1863, axis 1 0 0
- added joint mecanum_joint_1_6: type continuous, parent wheel_link_1, child mecanum_link_1_6, origin xyz=0.010659 -0.010659 0.023168 rpy=0.27635 0 -2.3562, axis 1 0 0
- added joint mecanum_joint_1_7: type continuous, parent wheel_link_1, child mecanum_link_1_7, origin xyz=-0.0088452 -0.010659 0.02392 rpy=-0.53767 0.5236 -2.1863, axis 1 0 0
- added joint mecanum_joint_1_8: type continuous, parent wheel_link_1, child mecanum_link_1_8, origin xyz=-0.0231684788371995 -0.0106594850812888 0.0106594850812885 rpy=-1.86346161677287 0.78539816339745 -1.57079632679489, axis 1 0 0
- added joint mecanum_joint_2_1: type continuous, parent wheel_link_2, child mecanum_link_2_1, origin xyz=0.021363 -0.17588 -0.011402 rpy=0.77425 -0.5236 0.95532, axis 1 0 0
- added joint mecanum_joint_2_2: type continuous, parent wheel_link_2, child mecanum_link_2_2, origin xyz=0.0151879353075897 -0.167731034854988 -0.0231684788372002 rpy=-0.376585891854111 0 0.785398163397447, axis 1 0 0
- added joint mecanum_joint_2_3: type continuous, parent wheel_link_2, child mecanum_link_2_3, origin xyz=-0.0040571 -0.16549 -0.028708 rpy=0.30982 0.5236 0.95532, axis 1 0 0
- added joint mecanum_joint_2_4: type continuous, parent wheel_link_2, child mecanum_link_2_4, origin xyz=-0.023168 -0.16725 -0.015674 rpy=0.51899 0.7854 1.5708, axis 1 0 0
- added joint mecanum_joint_2_5: type continuous, parent wheel_link_2, child mecanum_link_2_5, origin xyz=-0.02392 0.010659 0.0088452 rpy=-1.2312 0.5236 2.1863, axis 1 0 0
- added joint mecanum_joint_2_6: type continuous, parent wheel_link_2, child mecanum_link_2_6, origin xyz=0.00021712 -0.18314 0.023168 rpy=0.10747 0 2.3562, axis 1 0 0
- added joint mecanum_joint_2_7: type continuous, parent wheel_link_2, child mecanum_link_2_7, origin xyz=0.015658 -0.18189 0.017108 rpy=-0.15091 -0.5236 2.1863, axis 1 0 0
- added joint mecanum_joint_2_8: type continuous, parent wheel_link_2, child mecanum_link_2_8, origin xyz=0.023168 -0.18314 -0.00021712 rpy=0.037466 -0.7854 1.5708, axis 1 0 0
- added joint mecanum_joint_3_1: type continuous, parent wheel_link_3, child mecanum_link_3_1, origin xyz=-0.000217121321762817 -0.188799430199766 -0.0231684788371997 rpy=2.57018773993724 0 0.785398163397447, axis 1 0 0
- added joint mecanum_joint_3_2: type continuous, parent wheel_link_3, child mecanum_link_3_2, origin xyz=0.0172631017108847 -0.187337075147043 -0.0155020752802366 rpy=-0.0695016648418689 -0.523598775598295 0.955316618124504, axis 1 0 0
- added joint mecanum_joint_3_3: type continuous, parent wheel_link_3, child mecanum_link_3_3, origin xyz=0.0231684788371991 -0.188799430199766 -0.000217121321762305 rpy=-1.74486637658552 -0.78539816339745 1.57079632679489, axis 1 0 0
- added joint mecanum_joint_3_4: type continuous, parent wheel_link_3, child mecanum_link_3_4, origin xyz=-0.028379233364908 -0.1716164910008 0.00438594362621422 rpy=2.50619973205918 0.523598775598301 2.18627603546529, axis 1 0 0
- added joint mecanum_joint_3_5: type continuous, parent wheel_link_3, child mecanum_link_3_5, origin xyz=0.0114865015184892 -0.181658196272472 0.0212786754726319 rpy=-2.54970053621489 -0.523598775598301 2.18627603546528, axis 1 0 0
- added joint mecanum_joint_3_6: type continuous, parent wheel_link_3, child mecanum_link_3_6, origin xyz=-0.0156486881360898 -0.172933620741915 0.0231684788371995 rpy=-2.46220871219138 0 2.35619449019235, axis 1 0 0
- added joint mecanum_joint_3_7: type continuous, parent wheel_link_3, child mecanum_link_3_7, origin xyz=-0.0231684788372004 -0.1741732316202 -0.014409077257804 rpy=-1.44899159791202 0.785398163397451 1.57079632679491, axis 1 0 0
- added joint mecanum_joint_3_8: type continuous, parent wheel_link_3, child mecanum_link_3_8, origin xyz=-0.0114063522646582 -0.181544848110688 -0.0213588247264644 rpy=-2.70059865420832 0.523598775598307 0.955316618124512, axis 1 0 0
- added joint mecanum_joint_4_1: type continuous, parent wheel_link_4, child mecanum_link_4_1, origin xyz=-0.02392 -0.010659 -0.0088452 rpy=3.0576 0.5236 -0.95532, axis 1 0 0
- added joint mecanum_joint_4_2: type continuous, parent wheel_link_4, child mecanum_link_4_2, origin xyz=-0.010659 -0.010659 -0.023168 rpy=-1.6479 0 -0.7854, axis 1 0 0
- added joint mecanum_joint_4_3: type continuous, parent wheel_link_4, child mecanum_link_4_3, origin xyz=0.0088452 -0.010659 -0.02392 rpy=1.9316 -0.5236 -0.95532, axis 1 0 0
- added joint mecanum_joint_4_4: type continuous, parent wheel_link_4, child mecanum_link_4_4, origin xyz=0.023168 -0.010659 -0.010659 rpy=0.19357 -0.7854 -1.5708, axis 1 0 0
- added joint mecanum_joint_4_5: type continuous, parent wheel_link_4, child mecanum_link_4_5, origin xyz=0.02392 -0.010659 0.0088452 rpy=-2.5986 -0.5236 -2.1863, axis 1 0 0
- added joint mecanum_joint_4_6: type continuous, parent wheel_link_4, child mecanum_link_4_6, origin xyz=0.010659 -0.010659 0.023168 rpy=0.27635 0 -2.3562, axis 1 0 0
- added joint mecanum_joint_4_7: type continuous, parent wheel_link_4, child mecanum_link_4_7, origin xyz=-0.0088452 -0.010659 0.02392 rpy=-0.53767 0.5236 -2.1863, axis 1 0 0
- added joint mecanum_joint_4_8: type continuous, parent wheel_link_4, child mecanum_link_4_8, origin xyz=-0.0231684788371995 -0.0106594850812888 0.0106594850812885 rpy=-1.86346161677287 0.78539816339745 -1.57079632679489, axis 1 0 0
- joint wheel_joint_1: axis 0 0 1 -> 0 1 0; limit lower=-1.79769E+308 upper=1.79769E+308 effort=100 velocity=10 -> (none); origin xyz=0.0765 -0.0505 -0.0032237 rpy=1.5708 -1.179 -1.5708 -> xyz=0.0808 -0.25731 -0.0032237 rpy=1.5708 1.5708 3.1415
- joint wheel_joint_2: axis 0 0 1 -> 0 1 0; limit lower=-1.79769E+308 upper=1.79769E+308 effort=100 velocity=10 -> (none); origin xyz=-0.0765 -0.0505 -0.0032237 rpy=1.5708 1.179 1.5708 -> xyz=0.0808 -0.25731 -0.0032237 rpy=1.5708 -1.5708 3.1415
- joint wheel_joint_3: axis 0 0 1 -> 0 1 0; limit lower=-1.79769E+308 upper=1.79769E+308 effort=100 velocity=10 -> (none); origin xyz=-0.0765 -0.25731 -0.0032237 rpy=1.5708 -1.179 -1.5708 -> xyz=-0.0808 -0.0505 -0.0032237 rpy=1.5708 -1.5708 0
- joint wheel_joint_4: axis 0 0 1 -> 0 1 0; limit lower=-1.79769E+308 upper=1.79769E+308 effort=100 velocity=10 -> (none); origin xyz=0.0765 -0.25731 -0.0032237 rpy=1.5708 1.179 1.5708 -> xyz=-0.0808 -0.0505 -0.0032237 rpy=1.5708 -1.5708 3.1415

Commit message: fixed wheel 2 issue with wandering mecanum

File: robot_v3/urdf/model.urdf (robot description, URDF)
Before this commit: robot robot_v3, 43 links, 42 joints
Joints:
- joint mecanum_joint_2_1: origin xyz=0.021363 -0.17588 -0.011402 rpy=0.77425 -0.5236 0.95532 -> xyz=-0.000217121321762817 -0.188799430199766 -0.0231684788371997 rpy=2.57018773993724 0 0.785398163397447
- joint mecanum_joint_2_2: origin xyz=0.0151879353075897 -0.167731034854988 -0.0231684788372002 rpy=-0.376585891854111 0 0.785398163397447 -> xyz=0.0172631017108847 -0.187337075147043 -0.0155020752802366 rpy=-0.0695016648418689 -0.523598775598295 0.955316618124504
- joint mecanum_joint_2_3: origin xyz=-0.0040571 -0.16549 -0.028708 rpy=0.30982 0.5236 0.95532 -> xyz=0.0231684788371991 -0.188799430199766 -0.000217121321762305 rpy=-1.74486637658552 -0.78539816339745 1.57079632679489
- joint mecanum_joint_2_4: origin xyz=-0.023168 -0.16725 -0.015674 rpy=0.51899 0.7854 1.5708 -> xyz=-0.028379233364908 -0.1716164910008 0.00438594362621422 rpy=2.50619973205918 0.523598775598301 2.18627603546529
- joint mecanum_joint_2_5: origin xyz=-0.02392 0.010659 0.0088452 rpy=-1.2312 0.5236 2.1863 -> xyz=0.0114865015184892 -0.181658196272472 0.0212786754726319 rpy=-2.54970053621489 -0.523598775598301 2.18627603546528
- joint mecanum_joint_2_6: origin xyz=0.00021712 -0.18314 0.023168 rpy=0.10747 0 2.3562 -> xyz=-0.0156486881360898 -0.172933620741915 0.0231684788371995 rpy=-2.46220871219138 0 2.35619449019235
- joint mecanum_joint_2_7: origin xyz=0.015658 -0.18189 0.017108 rpy=-0.15091 -0.5236 2.1863 -> xyz=-0.0231684788372004 -0.1741732316202 -0.014409077257804 rpy=-1.44899159791202 0.785398163397451 1.57079632679491
- joint mecanum_joint_2_8: origin xyz=0.023168 -0.18314 -0.00021712 rpy=0.037466 -0.7854 1.5708 -> xyz=-0.0114063522646582 -0.181544848110688 -0.0213588247264644 rpy=-2.70059865420832 0.523598775598307 0.955316618124512
