Commit message: usind extern mecanum wheels

File: robot_v3/urdf/model.urdf (robot description, URDF)
Before this commit: robot robot_v3, 43 links, 42 joints
Links:
- removed link mecanum_link_1_1
- removed link mecanum_link_1_2
- removed link mecanum_link_1_3
- removed link mecanum_link_1_4
- removed link mecanum_link_1_5
- removed link mecanum_link_1_6
- removed link mecanum_link_1_7
- removed link mecanum_link_1_8
- removed link mecanum_link_2_1
- removed link mecanum_link_2_2
- removed link mecanum_link_2_3
- removed link mecanum_link_2_4
- removed link mecanum_link_2_5
- removed link mecanum_link_2_6
- removed link mecanum_link_2_7
- removed link mecanum_link_2_8
- removed link mecanum_link_3_1
- removed link mecanum_link_3_2
- removed link mecanum_link_3_3
- removed link mecanum_link_3_4
- removed link mecanum_link_3_5
- removed link mecanum_link_3_6
- removed link mecanum_link_3_7
- removed link mecanum_link_3_8
- removed link mecanum_link_4_1
- removed link mecanum_link_4_2
- removed link mecanum_link_4_3
- removed link mecanum_link_4_4
- removed link mecanum_link_4_5
- removed link mecanum_link_4_6
- removed link mecanum_link_4_7
- removed link mecanum_link_4_8
- removed link wheel_link_1
- removed link wheel_link_2
- removed link wheel_link_3
- removed link wheel_link_4
- added link roller_10_1, mass 0.014233736590696993; collision mesh filename=file://meshes/roller_10_1.stl scale=0.001 0.001 0.001; visual mesh filename=file://meshes/roller_10_1.stl scale=0.001 0.001 0.001
- added link roller_11_1, mass 0.014233736590697477; collision mesh filename=file://meshes/roller_11_1.stl scale=0.001 0.001 0.001; visual mesh filename=file://meshes/roller_11_1.stl scale=0.001 0.001 0.001
- added link roller_12_1, mass 0.01423373659069688; collision mesh filename=file://meshes/roller_12_1.stl scale=0.001 0.001 0.001; visual mesh filename=file://meshes/roller_12_1.stl scale=0.001 0.001 0.001
- added link roller_13_1, mass 0.014233736590696914; collision mesh filename=file://meshes/roller_13_1.stl scale=0.001 0.001 0.001; visual mesh filename=file://meshes/roller_13_1.stl scale=0.001 0.001 0.001
- added link roller_14_1, mass 0.014233736590697255; collision mesh filename=file://meshes/roller_14_1.stl scale=0.001 0.001 0.001; visual mesh filename=file://meshes/roller_14_1.stl scale=0.001 0.001 0.001
- added link roller_15_1, mass 0.014233736590697089; collision mesh filename=file://meshes/roller_15_1.stl scale=0.001 0.001 0.001; visual mesh filename=file://meshes/roller_15_1.stl scale=0.001 0.001 0.001
- added link roller_16_1, mass 0.01423373659069693; collision mesh filename=file://meshes/roller_16_1.stl scale=0.001 0.001 0.001; visual mesh filename=file://meshes/roller_16_1.stl scale=0.001 0.001 0.001
- added link roller_17_1, mass 0.014233736590697006; collision mesh filename=file://meshes/roller_17_1.stl scale=0.001 0.001 0.001; visual mesh filename=file://meshes/roller_17_1.stl scale=0.001 0.001 0.001
- added link roller_18_1, mass 0.01423373659069696; collision mesh filename=file://meshes/roller_18_1.stl scale=0.001 0.001 0.001; visual mesh filename=file://meshes/roller_18_1.stl scale=0.001 0.001 0.001
- added link roller_19_1, mass 0.014233736590697066; collision mesh filename=file://meshes/roller_19_1.stl scale=0.001 0.001 0.001; visual mesh filename=file://meshes/roller_19_1.stl scale=0.001 0.001 0.001
- added link roller_1_1, mass 0.014233736590697087; collision mesh filename=file://meshes/roller_1_1.stl scale=0.001 0.001 0.001; visual mesh filename=file://meshes/roller_1_1.stl scale=0.001 0.001 0.001
- added link roller_20_1, mass 0.014233736590696985; collision mesh filename=file://meshes/roller_20_1.stl scale=0.001 0.001 0.001; visual mesh filename=file://meshes/roller_20_1.stl scale=0.001 0.001 0.001
- added link roller_21_1, mass 0.014233736590696936; collision mesh filename=file://meshes/roller_21_1.stl scale=0.001 0.001 0.001; visual mesh filename=file://meshes/roller_21_1.stl scale=0.001 0.001 0.001
- added link roller_22_1, mass 0.014233736590697042; collision mesh filename=file://meshes/roller_22_1.stl scale=0.001 0.001 0.001; visual mesh filename=file://meshes/roller_22_1.stl scale=0.001 0.001 0.001
- added link roller_23_1, mass 0.014233736590696983; collision mesh filename=file://meshes/roller_23_1.stl scale=0.001 0.001 0.001; visual mesh filename=file://meshes/roller_23_1.stl scale=0.001 0.001 0.001
- added link roller_24_1, mass 0.014233736590697; collision mesh filename=file://meshes/roller_24_1.stl scale=0.001 0.001 0.001; visual mesh filename=file://meshes/roller_24_1.stl scale=0.001 0.001 0.001
- added link roller_25_1, mass 0.014233736590697047; collision mesh filename=file://meshes/roller_25_1.stl scale=0.001 0.001 0.001; visual mesh filename=file://meshes/roller_25_1.stl scale=0.001 0.001 0.001
- added link roller_26_1, mass 0.014233736590697033; collision mesh filename=file://meshes/roller_26_1.stl scale=0.001 0.001 0.001; visual mesh filename=file://meshes/roller_26_1.stl scale=0.001 0.001 0.001
- added link roller_27_1, mass 0.014233736590697002; collision mesh filename=file://meshes/roller_27_1.stl scale=0.001 0.001 0.001; visual mesh filename=file://meshes/roller_27_1.stl scale=0.001 0.001 0.001
- added link roller_28_1, mass 0.014233736590697; collision mesh filename=file://meshes/roller_28_1.stl scale=0.001 0.001 0.001; visual mesh filename=file://meshes/roller_28_1.stl scale=0.001 0.001 0.001
- added link roller_29_1, mass 0.014233736590697115; collision mesh filename=file://meshes/roller_29_1.stl scale=0.001 0.001 0.001; visual mesh filename=file://meshes/roller_29_1.stl scale=0.001 0.001 0.001
- added link roller_2_1, mass 0.014233736590697151; collision mesh filename=file://meshes/roller_2_1.stl scale=0.001 0.001 0.001; visual mesh filename=file://meshes/roller_2_1.stl scale=0.001 0.001 0.001
- added link roller_30_1, mass 0.014233736590697087; collision mesh filename=file://meshes/roller_30_1.stl scale=0.001 0.001 0.001; visual mesh filename=file://meshes/roller_30_1.stl scale=0.001 0.001 0.001
- added link roller_31_1, mass 0.01423373659069689; collision mesh filename=file://meshes/roller_31_1.stl scale=0.001 0.001 0.001; visual mesh filename=file://meshes/roller_31_1.stl scale=0.001 0.001 0.001
- added link roller_32_1, mass 0.014233736590697054; collision mesh filename=file://meshes/roller_32_1.stl scale=0.001 0.001 0.001; visual mesh filename=file://meshes/roller_32_1.stl scale=0.001 0.001 0.001
- added link roller_33_1, mass 0.01423373659069702; collision mesh filename=file://meshes/roller_33_1.stl scale=0.001 0.001 0.001; visual mesh filename=file://meshes/roller_33_1.stl scale=0.001 0.001 0.001
- added link roller_34_1, mass 0.014233736590696927; collision mesh filename=file://meshes/roller_34_1.stl scale=0.001 0.001 0.001; visual mesh filename=file://meshes/roller_34_1.stl scale=0.001 0.001 0.001
- added link roller_35_1, mass 0.01423373659069706; collision mesh filename=file://meshes/roller_35_1.stl scale=0.001 0.001 0.001; visual mesh filename=file://meshes/roller_35_1.stl scale=0.001 0.001 0.001
- added link roller_36_1, mass 0.014233736590696964; collision mesh filename=file://meshes/roller_36_1.stl scale=0.001 0.001 0.001; visual mesh filename=file://meshes/roller_36_1.stl scale=0.001 0.001 0.001
- added link roller_3_1, mass 0.014233736590696551; collision mesh filename=file://meshes/roller_3_1.stl scale=0.001 0.001 0.001; visual mesh filename=file://meshes/roller_3_1.stl scale=0.001 0.001 0.001
- added link roller_4_1, mass 0.01423373659069714; collision mesh filename=file://meshes/roller_4_1.stl scale=0.001 0.001 0.001; visual mesh filename=file://meshes/roller_4_1.stl scale=0.001 0.001 0.001
- added link roller_5_1, mass 0.01423373659069685; collision mesh filename=file://meshes/roller_5_1.stl scale=0.001 0.001 0.001; visual mesh filename=file://meshes/roller_5_1.stl scale=0.001 0.001 0.001
- added link roller_6_1, mass 0.014233736590697; collision mesh filename=file://meshes/roller_6_1.stl scale=0.001 0.001 0.001; visual mesh filename=file://meshes/roller_6_1.stl scale=0.001 0.001 0.001
- added link roller_7_1, mass 0.014233736590697038; collision mesh filename=file://meshes/roller_7_1.stl scale=0.001 0.001 0.001; visual mesh filename=file://meshes/roller_7_1.stl scale=0.001 0.001 0.001
- added link roller_8_1, mass 0.01423373659069701; collision mesh filename=file://meshes/roller_8_1.stl scale=0.001 0.001 0.001; visual mesh filename=file://meshes/roller_8_1.stl scale=0.001 0.001 0.001
- added link roller_9_1, mass 0.014233736590696988; collision mesh filename=file://meshes/roller_9_1.stl scale=0.001 0.001 0.001; visual mesh filename=file://meshes/roller_9_1.stl scale=0.001 0.001 0.001
- added link wheel_frame_BL_1, mass 0.30282113324994536; collision mesh filename=file://meshes/wheel_frame_BL_1.stl scale=0.001 0.001 0.001; visual mesh filename=file://meshes/wheel_frame_BL_1.stl scale=0.001 0.001 0.001
- added link wheel_frame_BR_1, mass 0.30282113324994864; collision mesh filename=file://meshes/wheel_frame_BR_1.stl scale=0.001 0.001 0.001; visual mesh filename=file://meshes/wheel_frame_BR_1.stl scale=0.001 0.001 0.001
- added link wheel_frame_FL_1, mass 0.30282113324994747; collision mesh filename=file://meshes/wheel_frame_FL_1.stl scale=0.001 0.001 0.001; visual mesh filename=file://meshes/wheel_frame_FL_1.stl scale=0.001 0.001 0.001
- added link wheel_frame_FR_1, mass 0.30282113324994836; collision mesh filename=file://meshes/wheel_frame_FR_1.stl scale=0.001 0.001 0.001; visual mesh filename=file://meshes/wheel_frame_FR_1.stl scale=0.001 0.001 0.001
- link aruco_link: mass 8.1643 -> 0.001
- link base_link: mass 8.1643 -> 18.1643
Joints:
- removed joint mecanum_joint_1_1
- removed joint mecanum_joint_1_2
- removed joint mecanum_joint_1_3
- removed joint mecanum_joint_1_4
- removed joint mecanum_joint_1_5
- removed joint mecanum_joint_1_6
- removed joint mecanum_joint_1_7
- removed joint mecanum_joint_1_8
- removed joint mecanum_joint_2_1
- removed joint mecanum_joint_2_2
- removed joint mecanum_joint_2_3
- removed joint mecanum_joint_2_4
- removed joint mecanum_joint_2_5
- removed joint mecanum_joint_2_6
- removed joint mecanum_joint_2_7
- removed joint mecanum_joint_2_8
- removed joint mecanum_joint_3_1
- removed joint mecanum_joint_3_2
- removed joint mecanum_joint_3_3
- removed joint mecanum_joint_3_4
- removed joint mecanum_joint_3_5
- removed joint mecanum_joint_3_6
- removed joint mecanum_joint_3_7
- removed joint mecanum_joint_3_8
- removed joint mecanum_joint_4_1
- removed joint mecanum_joint_4_2
- removed joint mecanum_joint_4_3
- removed joint mecanum_joint_4_4
- removed joint mecanum_joint_4_5
- removed joint mecanum_joint_4_6
- removed joint mecanum_joint_4_7
- removed joint mecanum_joint_4_8
- added joint Revolute_57: type continuous, parent wheel_frame_FL_1, child roller_14_1, origin xyz=0.017316 -0.007119 0.04 rpy=0 0 0, axis 0.720551 0.693402 -0.0
- added joint Revolute_58: type continuous, parent wheel_frame_FL_1, child roller_16_1, origin xyz=0.038976 -0.007119 0.019512 rpy=0 0 0, axis 0.551974 0.693402 -0.463161
- added joint Revolute_59: type continuous, parent wheel_frame_FL_1, child roller_13_1, origin xyz=0.042394 -0.007086 -0.010075 rpy=0 0 0, axis -0.125122 -0.693402 0.709604
- added joint Revolute_60: type continuous, parent wheel_frame_FL_1, child roller_12_1, origin xyz=0.025999 -0.007086 -0.034968 rpy=0 0 0, axis 0.360276 -0.693402 0.624016
- added joint Revolute_61: type continuous, parent wheel_frame_FL_1, child roller_15_1, origin xyz=-0.00256 -0.007086 -0.043499 rpy=0 0 0, axis 0.677097 -0.693402 0.246443
- added joint Revolute_62: type continuous, parent wheel_frame_FL_1, child roller_17_1, origin xyz=-0.029922 -0.007086 -0.031676 rpy=0 0 0, axis 0.677097 -0.693402 -0.246443
- added joint Revolute_63: type continuous, parent wheel_frame_FL_1, child roller_18_1, origin xyz=-0.043283 -0.007086 -0.005032 rpy=0 0 0, axis 0.360276 -0.693402 -0.624016
- added joint Revolute_64: type continuous, parent wheel_frame_FL_1, child roller_10_1, origin xyz=-0.036391 -0.007086 0.023967 rpy=0 0 0, axis -0.125122 -0.693402 -0.709604
- added joint Revolute_65: type continuous, parent wheel_frame_FL_1, child roller_11_1, origin xyz=-0.012472 -0.007086 0.041751 rpy=0 0 0, axis -0.551974 -0.693402 -0.463161
- added joint Revolute_67: type continuous, parent wheel_frame_FR_1, child roller_7_1, origin xyz=-0.017316 0.040381 0.04 rpy=0 0 0, axis 0.720551 -0.693402 -0.0
- added joint Revolute_68: type continuous, parent wheel_frame_FR_1, child roller_5_1, origin xyz=0.012447 0.040381 0.041772 rpy=0 0 0, axis 0.551974 -0.693402 -0.463161
- added joint Revolute_69: type continuous, parent wheel_frame_FR_1, child roller_3_1, origin xyz=0.036385 0.040381 0.023998 rpy=0 0 0, axis 0.125122 -0.693402 -0.709604
- added joint Revolute_70: type continuous, parent wheel_frame_FR_1, child roller_6_1, origin xyz=0.043299 0.040381 -0.005004 rpy=0 0 0, axis -0.360276 -0.693402 -0.624016
- added joint Revolute_71: type continuous, parent wheel_frame_FR_1, child roller_8_1, origin xyz=0.029952 0.040381 -0.031665 rpy=0 0 0, axis -0.677097 -0.693402 -0.246443
- added joint Revolute_72: type continuous, parent wheel_frame_FR_1, child roller_9_1, origin xyz=0.002591 0.040381 -0.04351 rpy=0 0 0, axis -0.677097 -0.693402 0.246443
- added joint Revolute_73: type continuous, parent wheel_frame_FR_1, child roller_4_1, origin xyz=-0.025983 0.040381 -0.034996 rpy=0 0 0, axis -0.360276 -0.693402 0.624016
- added joint Revolute_74: type continuous, parent wheel_frame_FR_1, child roller_1_1, origin xyz=-0.042399 0.040381 -0.010107 rpy=0 0 0, axis 0.125122 -0.693402 0.709604
- added joint Revolute_75: type continuous, parent wheel_frame_FR_1, child roller_2_1, origin xyz=-0.038976 0.040381 0.019512 rpy=0 0 0, axis 0.551974 -0.693402 0.463161
- added joint Revolute_77: type continuous, parent wheel_frame_BL_1, child roller_23_1, origin xyz=-0.017316 -0.007119 0.04 rpy=0 0 0, axis 0.720551 -0.693402 -0.0
- added joint Revolute_78: type continuous, parent wheel_frame_BL_1, child roller_22_1, origin xyz=0.012447 -0.007119 0.041772 rpy=0 0 0, axis 0.551974 -0.693402 -0.463161
- added joint Revolute_79: type continuous, parent wheel_frame_BL_1, child roller_25_1, origin xyz=0.036385 -0.007119 0.023998 rpy=0 0 0, axis 0.125122 -0.693402 -0.709604
- added joint Revolute_80: type continuous, parent wheel_frame_BL_1, child roller_21_1, origin xyz=0.043299 -0.007119 -0.005004 rpy=0 0 0, axis -0.360276 -0.693402 -0.624016
- added joint Revolute_81: type continuous, parent wheel_frame_BL_1, child roller_26_1, origin xyz=0.029952 -0.007119 -0.031665 rpy=0 0 0, axis -0.677097 -0.693402 -0.246443
- added joint Revolute_82: type continuous, parent wheel_frame_BL_1, child roller_27_1, origin xyz=0.002591 -0.007119 -0.04351 rpy=0 0 0, axis -0.677097 -0.693402 0.246443
- added joint Revolute_83: type continuous, parent wheel_frame_BL_1, child roller_20_1, origin xyz=-0.025983 -0.007119 -0.034996 rpy=0 0 0, axis -0.360276 -0.693402 0.624016
- added joint Revolute_84: type continuous, parent wheel_frame_BL_1, child roller_19_1, origin xyz=-0.042399 -0.007119 -0.010107 rpy=0 0 0, axis 0.125122 -0.693402 0.709604
- added joint Revolute_85: type continuous, parent wheel_frame_BL_1, child roller_24_1, origin xyz=-0.038976 -0.007119 0.019512 rpy=0 0 0, axis 0.551974 -0.693402 0.463161
- added joint Revolute_87: type continuous, parent wheel_frame_BR_1, child roller_34_1, origin xyz=0.017316 0.040381 0.04 rpy=0 0 0, axis 0.720551 0.693402 -0.0
- added joint Revolute_88: type continuous, parent wheel_frame_BR_1, child roller_30_1, origin xyz=0.038976 0.040381 0.019512 rpy=0 0 0, axis 0.551974 0.693402 -0.463161
- added joint Revolute_89: type continuous, parent wheel_frame_BR_1, child roller_32_1, origin xyz=0.042399 0.040381 -0.010107 rpy=0 0 0, axis 0.125122 0.693402 -0.709604
- added joint Revolute_90: type continuous, parent wheel_frame_BR_1, child roller_31_1, origin xyz=0.025983 0.040381 -0.034996 rpy=0 0 0, axis -0.360276 0.693402 -0.624016
- added joint Revolute_91: type continuous, parent wheel_frame_BR_1, child roller_29_1, origin xyz=-0.002591 0.040381 -0.04351 rpy=0 0 0, axis -0.677097 0.693402 -0.246443
- added joint Revolute_92: type continuous, parent wheel_frame_BR_1, child roller_28_1, origin xyz=-0.012447 0.040381 0.041772 rpy=0 0 0, axis 0.551974 0.693402 0.463161
- added joint Revolute_93: type continuous, parent wheel_frame_BR_1, child roller_35_1, origin xyz=-0.029952 0.040381 -0.031665 rpy=0 0 0, axis -0.677097 0.693402 0.246443
- added joint Revolute_94: type continuous, parent wheel_frame_BR_1, child roller_36_1, origin xyz=-0.043299 0.040381 -0.005004 rpy=0 0 0, axis -0.360276 0.693402 0.624016
- added joint Revolute_95: type continuous, parent wheel_frame_BR_1, child roller_33_1, origin xyz=-0.036391 0.040414 0.023967 rpy=0 0 0, axis -0.125122 -0.693402 -0.709604
- joint wheel_joint_1: child wheel_link_1 -> wheel_frame_BR_1; origin xyz=0.0808 -0.25731 -0.0032237 rpy=1.5708 1.5708 3.1415 -> xyz=0.0808 -0.25731 -0.0032237 rpy=1.5708 1.5708 0
- joint wheel_joint_2: child wheel_link_2 -> wheel_frame_BL_1; origin xyz=0.0808 -0.25731 -0.0032237 rpy=1.5708 -1.5708 3.1415 -> xyz=-0.0808 -0.25731 -0.0032237 rpy=1.5708 -1.5708 3.1415
- joint wheel_joint_3: child wheel_link_3 -> wheel_frame_FR_1; origin xyz=-0.0808 -0.0505 -0.0032237 rpy=1.5708 -1.5708 0 -> xyz=0.0808 -0.0505 -0.0032237 rpy=1.5708 -1.5708 3.1415
- joint wheel_joint_4: child wheel_link_4 -> wheel_frame_FL_1

Commit message: working state

File: robot_v3/urdf/model.urdf (robot description, URDF)
Before this commit: robot robot_v3, 47 links, 46 joints
Links:
- removed link link_1
- removed link link_2
- removed link link_3
- removed link link_4
- removed link pre_link_5
Joints:
- removed joint joint_1
- removed joint joint_2
- removed joint joint_3
- removed joint joint_4
- removed joint joint_5
- joint joint_aruco_tag: origin xyz=0.0 -0.22 0.051 rpy=0 0 0 -> xyz=0.0 -0.22 0.101 rpy=0 0 3.1415

Commit message: somewhat working but very slow

File: robot_v3/urdf/model.urdf (robot description, URDF)
Before this commit: robot robot_v3, 42 links, 41 joints
Links:
- added link link_1, mass 3.16; collision mesh filename=file://meshes/link_1.STL; visual mesh filename=file://meshes/link_1.STL
- added link link_2, mass 0.22008; collision mesh filename=file://meshes/link_2.STL; visual mesh filename=file://meshes/link_2.STL
- added link link_3, mass 0.11515; collision mesh filename=file://meshes/link_3.STL; visual mesh filename=file://meshes/link_3.STL
- added link link_4, mass 0.11556; collision mesh filename=file://meshes/link_4.STL; visual mesh filename=file://meshes/link_4.STL
- added link pre_link_5, mass 0.0010902; collision mesh filename=file://meshes/pre_link_5.STL; visual mesh filename=file://meshes/pre_link_5.STL
Joints:
- added joint joint_1: type continuous, parent base_link, child link_1, origin xyz=0 -0.081313 0.08128 rpy=-1.5708 0 -3.1416, axis 0 1 0, limit lower=-3.1415 upper=3.1415 effort=100 velocity=5
- added joint joint_2: type continuous, parent link_1, child link_2, origin xyz=0 -0.024358 0.0098714 rpy=-1.5708 0 3.1416, axis 1 0 0, limit lower=-3.1415 upper=3.1415 effort=100 velocity=5
- added joint joint_3: type continuous, parent link_2, child link_3, origin xyz=0 -0.13432 0 rpy=3.1416 0 0, axis 1 0 0, limit lower=-3.1415 upper=3.1415 effort=100 velocity=5
- added joint joint_4: type continuous, parent link_3, child link_4, origin xyz=0 0 -0.087743 rpy=3.1416 0 0, axis 1 0 0, limit lower=-3.1415 upper=3.1415 effort=100 velocity=5
- added joint joint_5: type continuous, parent link_4, child pre_link_5, origin xyz=-0.00060377 0.00065019 0.063746 rpy=-1.5708 0 0.59278, axis 0 1 0, limit lower=-3.1415 upper=3.1415 effort=100 velocity=5
